File: float_pcb.kicad_pcb (KiCad board)
At the start: 2 copper layers, 71 x 41.5 mm, 37 parts, among them J1 BR Switch, J2 5V, J3 USB_C, J4 Servo, Q1 Q_PMOS_GSD, SW1 SW_Push, SW2 SW_Push, U1 TPSM863252RDXR, U2 TPSM863252RDXR, U3 ESP32-S3-MINI-1U

Commit message: more changes
Parts:
- removed BT1: 7.4V, Connector_AMASS:AMASS_XT30U-F_1x02_P5.0mm_Vertical
- removed C11: .1uF, Capacitor_SMD:C_0805_2012Metric
- removed F1: 5A, Fuse:Fuseholder_Cylinder-5x20mm_Schurter_0031_8201_Horizontal_Open
- removed SW1: SW_Push, Button_Switch_SMD:SW_SPST_TL3342
- removed U1, U2: TPSM863252RDXR, TPSM863252RDXR:RDX0007A-MFG
- added D1: BATT_STAT, LED_SMD:LED_0805_2012Metric, F.Cu at (101.5, 89.5)
- added D2: LED, LED_SMD:LED_0805_2012Metric, F.Cu at (120.9, 66.8)
- added D3: LED, LED_SMD:LED_0805_2012Metric, F.Cu at (120.9, 69.9)
- added J5: BR_DEPTH_SENSOR, Connector_JST:JST_GH_BM04B-GHS-TBT_1x04-1MP_P1.25mm_Vertical, F.Cu at (111.7, 75.4)
- added J6: BR Light, Connector_JST:JST_VH_B2P-VH_1x02_P3.96mm_Vertical, F.Cu at (126.5, 67.0)
- added J7: Batt, Connector_AMASS:AMASS_XT30U-M_1x02_P5.0mm_Vertical, F.Cu at (99.0, 67.0)
- added R14: 2.7kQ, Resistor_SMD:R_0805_2012Metric, F.Cu at (95.5, 89.5)
- added R15: 650Q, Resistor_SMD:R_0805_2012Metric, F.Cu at (116.4, 72.6)
- added R16: 1.5kQ, LED_SMD:LED_0805_2012Metric, F.Cu at (120.9, 72.9)
- added R17: 10kQ, Resistor_SMD:R_0805_2012Metric, F.Cu at (116.4, 75.5)
- added R18: R, Resistor_SMD:R_0805_2012Metric, F.Cu at (114.2, 92.5)
- added R19: R, Resistor_SMD:R_0805_2012Metric, F.Cu at (115.5, 99.0)
- added SW3: ENABLE, Button_Switch_SMD:SW_SPST_TL3342, F.Cu at (135.0, 56.5)
- added VR1: TPSM863252RDXR, TPSM863252RDXR:VREG_TPSM863252RDXR, F.Cu at (127.7, 94.5)
- added VR2: TPSM863252RDXR, TPSM863252RDXR:VREG_TPSM863252RDXR, F.Cu at (109.8, 97.3)
- C12: value .1uF -> 1uF
- J4: value Servo -> Conn_01x02; footprint Connector_PinHeader_2.54mm:PinHeader_1x01_P2.54mm_Vertical -> Connector_PinHeader_2.54mm:PinHeader_1x02_P2.54mm_Vertical
- Q1: value Q_PMOS_GSD -> AO3400A; footprint Package_TO_SOT_SMD:SOT-223-3_TabPin2 -> Package_TO_SOT_SMD:SOT-23
- R1: value 100kQ -> 4.7kQ
- R13: value 10kQ -> 4.7kQ
- moved C12 51.9 mm to (110.1, 62.5), turned to 0 degrees
- moved R12 50.6 mm to (110.1, 65.5), turned to 0 degrees
- moved R1 39.1 mm to (116.4, 63.8), turned to 0 degrees
- moved Q1 29.6 mm to (125.5, 75.0), turned to 0 degrees
- moved C9 22.5 mm to (115.0, 95.3), turned to 90 degrees
- moved J4 21.9 mm to (160.0, 68.5)
- moved R13 20.8 mm to (116.4, 66.7), turned to 0 degrees
- moved C6 18.2 mm to (94.5, 95.5)
- moved C7 17.7 mm to (99.5, 95.5)
- moved C8 17.4 mm to (110.0, 91.0), turned to 0 degrees
- moved R6 17.1 mm to (105.0, 93.0)
- moved R7 17.0 mm to (105.0, 98.0)
- moved J1 7.47 mm to (99.0, 80.5), turned to -90 degrees
- moved C2 6.29 mm to (108.5, 84.0)
Connections:
- C1 pad 1: Net-(Q1-G) -> +BATT
- C2 pad 1: Net-(Q1-G) -> +BATT
- C4 pad 1: Net-(U1-VOUT) -> +3V3
- C5 pad 1: Net-(U1-VOUT) -> +3V3
- C6 pad 1: Net-(Q1-G) -> +BATT
- C7 pad 1: Net-(Q1-G) -> +BATT
- J1 pad 2: Net-(J1-Pin_2) -> +BATT
- Q1 pad 1: Net-(Q1-G) -> LIGHT
- Q1 pad 2: Net-(Q1-G) -> GND
- Q1 pad 3: Net-(J1-Pin_2) -> Net-(J6-Pin_2)
- R1 pad 1: Net-(Q1-G) -> +3V3
- R1 pad 2: GND -> /SCL
- R12 pad 1: Net-(U1-VOUT) -> +3V3
- R13 pad 1: Net-(U1-VOUT) -> /SDA
- R13 pad 2: Net-(U3-IO0) -> +3V3
- R2 pad 1: Net-(Q1-G) -> +BATT
- R4 pad 1: Net-(U1-VOUT) -> +3V3
- R6 pad 1: Net-(Q1-G) -> +BATT
- U3 pad 16: unconnected-(U3-IO12-Pad16) -> /SCL
- U3 pad 17: unconnected-(U3-IO13-Pad17) -> /SDA
- U3 pad 21: Net-(J4-Pin_1) -> Net-(J4-Pin_2)
- U3 pad 22: unconnected-(U3-IO18-Pad22) -> Net-(J4-Pin_1)
- U3 pad 3: Net-(U1-VOUT) -> +3V3
- U3 pad 37: unconnected-(U3-IO41-Pad37) -> LIGHT
Routing:
- net Net-(U1-VOUT): track 64.9 -> 0.00 mm, vias 4 -> 0
- net Net-(Q1-G): track 58.1 -> 0.00 mm
- net Net-(U3-EN): track 47.2 -> 0.00 mm
- net +BATT: track 0.00 -> 28.8 mm
- net Net-(C4-Pad2): track 28.2 -> 0.00 mm
- net Net-(J2-Pin_1): track 27.8 -> 0.00 mm
- net Net-(U3-USB_D-): track 22.4 -> 0.00 mm, vias 2 -> 0
- net Net-(J1-Pin_1): track 30.1 -> 8.56 mm
- net Net-(U3-USB_D+): track 20.6 -> 0.00 mm
- net Net-(U3-IO0): track 19.0 -> 0.00 mm
- net Net-(BT1-+): track 14.4 -> 0.00 mm
- net Net-(J1-Pin_2): track 9.78 -> 0.00 mm
- net Net-(C9-Pad2): track 9.16 -> 0.00 mm
- net Net-(J4-Pin_1): track 5.47 -> 0.00 mm
- net unconnected-(VR2-PG-Pad5): track 0.00 -> 5.28 mm
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