File: float_pcb.kicad_pcb (KiCad board)
At the start: 4 copper layers, 64 x 64 mm, 68 parts, among them J1 Switch, J2 Conn_01x04, J3 USB_C, J4 Conn_01x03, J5 I2C, J6 Light, J7 Batt, J9 I2C, Q1 AO3400A, Q2 AO3400A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

Commit message: Progress
Parts:
- added R26: OPT, Resistor_SMD:R_0603_1608Metric, F.Cu at (170.0, 116.5)
- added TP10: EN, TestPoint:TestPoint_Pad_D1.5mm, B.Cu at (131.0, 108.8)
- added TP5: SCL2, TestPoint:TestPoint_Pad_D1.5mm, B.Cu at (152.5, 134.0)
- added TP6: SDA2, TestPoint:TestPoint_Pad_D1.5mm, B.Cu at (157.5, 128.0)
- added TP7: SDA2, TestPoint:TestPoint_Pad_D1.5mm, B.Cu at (143.5, 134.0)
- added TP8: SCL1, TestPoint:TestPoint_Pad_D1.5mm, B.Cu at (138.5, 128.0)
- added TP9: BOOT, TestPoint:TestPoint_Pad_D1.5mm, B.Cu at (175.5, 112.0)
- TP1, TP2, TP3, TP4: moved to B.Cu
- moved TP4 34.8 mm to (153.5, 83.5), turned to 180 degrees
- moved TP2 32.2 mm to (148.0, 130.5), turned to 180 degrees
- moved TP1 25.3 mm to (174.0, 101.0), turned to 180 degrees
- moved TP3 19.3 mm to (137.0, 115.5), turned to 180 degrees
- moved H1 1.35 mm to (126.5, 95.0)
- moved H2 1.27 mm to (174.0, 117.5)
- moved Q2 0.56 mm to (161.2, 117.0)
- moved R20 0.50 mm to (157.2, 117.0)
- moved J9 0.25 mm to (160.0, 130.5)
- moved R22 0.05 mm to (161.0, 105.5)
- moved R23 0.05 mm to (164.0, 102.5)
- moved R24 0.05 mm to (164.0, 112.0)
- moved R25 0.05 mm to (161.0, 109.0)
- moved U6 0.05 mm to (165.2, 107.2)
Connections:
- LS1 pad P: +3V3 -> Net-(LS1-PadP)
- TP2 pad 1: Net-(U1-VOUT) -> +3V3
- U4 pad 35: SERVO -> unconnected-(U4-IO42-Pad35)
- U4 pad 39: unconnected-(U4-IO1-Pad39) -> SERVO
Routing:
- net Net-(U4-IO0): track 6.30 -> 28.8 mm, vias 0 -> 1
- net Net-(J4-Pin_2): track 25.1 -> 32.8 mm
- net Net-(LS1-PadP): track 0.00 -> 5.90 mm
- net Net-(U1-VOUT): track 13.8 -> 19.7 mm
- net SCL2: track 24.5 -> 29.1 mm
- net SDA1: track 25.7 -> 30.2 mm
- net +BATT: track 72.6 -> 77.0 mm
- net +3V3: track 26.0 -> 30.0 mm, vias 14 -> 16
- net Net-(U4-EN): track 29.2 -> 32.7 mm
- net SCL1: track 22.7 -> 25.3 mm
- net SDA2: track 21.6 -> 24.1 mm
- net SERVO: track 11.3 -> 9.15 mm
- net GND: track 5.45 -> 7.02 mm
- net Net-(U2-EN): track 16.4 -> 15.7 mm
- net BUZZER: track 8.02 -> 7.46 mm
Other:
- board text added: "3V3 LINK"
- board text added: "BATT"
- board text added: "BOOT"
- board text added: "DATA ONLY"
- board text added: "EN"
- board text added: "SCL1"
- board text added: "SCL2"
- board text added: "SDA1"
- board text added: "SDA2"
- board text added: "SWITCH"

Commit message: Almost done with V4
Parts:
- added G***: LOGO, LOGO, B.Cu at (148.5, 99.2)
- added G***: LOGO, LOGO, B.Cu at (148.5, 115.2)
- R26: value OPT -> TBD
- moved TP3 9.82 mm to (127.5, 118.0)
- moved TP10 4.78 mm to (127.5, 112.0)
Routing:
- net GND: track 7.02 -> 9.77 mm
Other:
- board text added: "Evan Kim '27"
- board text added: "MISC"
- board text added: "REV A"
- board text removed: "DBG"
