File: float_pcb.kicad_sch (KiCad schematic)
At the start: 34 parts, among them J1 BR Switch, J2 5V, J3 USB_C, J4 Servo, SW2 SW_Push, SW3 ENABLE, U1 TPSM863252RDXR, U2 TPSM863252RDXR, U3 ESP32-S3-MINI-1U

Commit message: Add some things
Parts:
- added D1: BATT_STATUS, symbol Device:LED
- added D2, D3: LED, symbol Device:LED
- added J5: BR_DEPTH_SENSOR, Connector_JST:JST_GH_BM03B-GHS-TBT_1x03-1MP_P1.25mm_Vertical, symbol Connector_Generic:Conn_01x04
- added R1, R13: 4.7kQ, symbol Device:R
- added R14: 2.7kQ, symbol Device:R
- added R15: 650Q, symbol Device:R
- added R16: 1.5kQ, symbol Device:R
Connections:
- net +3.3V: now also R15.1
- net GND: now also D1.1 (K), D2.1 (K), D3.1 (K), J5.1 (Pin_1)
- net at C10.1, C9.1, J2.1 (Pin_1)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: now also R16.1
- net at F1.2, J1.1 (Pin_1): now also R14.2
- net SCL: now reaches U3.16 (IO12)
- net SCL: now also J5.3 (Pin_3), R1.2
- net SDA: now reaches U3.17 (IO13)
- net SDA: now also J5.2 (Pin_2), R13.1
- new net: D3.2 (A), R16.2
- new net: D2.2 (A), R15.2
- new net: D1.2 (A), R14.1
- new net +3V3: J5.4 (Pin_4), R1.1, R13.2
- no-connect marks 43 -> 40
Other:
- moved on the sheet: C10, J1, J4

Commit message: more changes
Parts:
- removed BT1: 7.4V, Connector_AMASS:AMASS_XT30U-F_1x02_P5.0mm_Vertical, symbol Device:Battery
- removed C11: .1uF, Capacitor_SMD:C_0805_2012Metric, symbol Device:C
- removed F1: 5A, Fuse:Fuseholder_Cylinder-5x20mm_Schurter_0031_8201_Horizontal_Open, symbol Device:Fuse
- removed J4: Servo, Connector_PinHeader_2.54mm:PinHeader_1x01_P2.54mm_Vertical, symbol Connector_Generic:Conn_01x01
- removed U1, U2: TPSM863252RDXR, TPSM863252RDXR:RDX0007A-MFG, symbol TPSM863252RDXR:TPSM863252RDXR
- added J4: Conn_01x02, Connector_PinHeader_2.54mm:PinHeader_1x02_P2.54mm_Vertical, symbol Connector_Generic:Conn_01x02
- added J6: BR Light, Connector_JST:JST_VH_B2P-VH_1x02_P3.96mm_Vertical, symbol Connector_Generic:Conn_01x02
- added J7: Batt, Connector_AMASS:AMASS_XT30U-M_1x02_P5.0mm_Vertical, symbol Connector_Generic:Conn_01x02
- added Q1: AO3400A, Package_TO_SOT_SMD:SOT-23, symbol Transistor_FET:AO3400A
- added R17: 10kQ, Resistor_SMD:R_0805_2012Metric, symbol Device:R
- added R18, R19: R, Resistor_SMD:R_0805_2012Metric, symbol Device:R
- added VR1, VR2: TPSM863252RDXR, TPSM863252RDXR:VREG_TPSM863252RDXR, symbol TPSM863252RDXR:TPSM863252RDXR
- D1: value BATT_STATUS -> BATT_STAT; footprint (none) -> LED_SMD:LED_0805_2012Metric
- D2, D3, R16: footprint (none) -> LED_SMD:LED_0805_2012Metric
- J5: footprint Connector_JST:JST_GH_BM03B-GHS-TBT_1x03-1MP_P1.25mm_Vertical -> Connector_JST:JST_GH_BM04B-GHS-TBT_1x04-1MP_P1.25mm_Vertical
- R1, R13, R14, R15: footprint (none) -> Resistor_SMD:R_0805_2012Metric
Connections:
- net +3.3V is gone; now on net +3V3: C4.1, C5.1, R12.1, R15.1, R4.1
- net +3V3: now also U3.3 (3V3), J6.1 (Pin_1), VR1.3 (VOUT)
- net +BATT: now also R14.2, VR1.1 (VIN), VR2.1 (VIN)
- net GND: now also J7.1 (Pin_1), Q1.2 (S), R17.1, VR1.4 (PGND), VR2.4 (PGND)
- net at C8.1: now also VR2.6 (EN)
- net at J1.1 (Pin_1): now also J7.2 (Pin_2); no longer R14.2
- net at C3.1: now also VR1.6 (EN)
- net at U3.21 (IO17): now also J4.2 (Pin_2)
- net at U3.22 (IO18): now also J4.1 (Pin_1)
- net LIGHT: now reaches U3.37 (IO41)
- net LIGHT: now also Q1.1 (G), R17.2
- new net: R19.1, VR2.3 (VOUT)
- new net: R18.2, VR1.7 (FB)
- new net: J6.2 (Pin_2), Q1.3 (D)
- no-connect marks 40 -> 38
Other:
- moved on the sheet: D1, R14
