File: float_pcb.kicad_sch (KiCad schematic)
At the start: 67 parts, among them J1 Switch, J2 Conn_01x04, J3 USB_C, J4 Conn_01x03, J5 I2C, J6 Light, J7 Batt, J9 I2C, Q1 AO3400A, Q2 AO3400A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

Commit message: Progress
Parts:
- added R26: OPT, Resistor_SMD:R_0603_1608Metric, symbol Device:R
- added TP10: EN, TestPoint:TestPoint_Pad_D1.5mm, symbol Connector:TestPoint
- added TP5: SCL2, TestPoint:TestPoint_Pad_D1.5mm, symbol Connector:TestPoint
- added TP6, TP7: SDA2, TestPoint:TestPoint_Pad_D1.5mm, symbol Connector:TestPoint
- added TP8: SCL1, TestPoint:TestPoint_Pad_D1.5mm, symbol Connector:TestPoint
- added TP9: BOOT, TestPoint:TestPoint_Pad_D1.5mm, symbol Connector:TestPoint
Connections:
- net +3V3: now also TP2.1, R26.2; no longer LS1.P
- net SCL1: now also TP8.1
- net SCL2: now also TP5.1
- net SDA1: now also TP7.1
- net SDA2: now also TP6.1
- net SERVO: now also U4.39 (IO1); no longer U4.35 (IO42)
- net at C4.1, C5.2, R15.2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: no longer TP2.1
- net at C12.2, ENABLE1.2, R12.2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: now also TP10.1
- net at BOOT1.1, U4.27 (IO0): now also TP9.1
- new net: LS1.P, R26.1
Other:
- note added: "Blue Robotics Light (Built-in Resistor)"
- note added: "Debug Plugs"
- note added: "ESD Protection"
- note removed: "Blue Robotics Light"
- moved on the sheet: BOOT1, C10, C2, C3, C4, C5, C6, C7, C8, C9, D2, D3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

Commit message: Almost done with V4
Parts:
- R26: value OPT -> TBD
Changed lines of the file:
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@@
 	)
 	(junction
-		(at 237.49 102.87)
-		(diameter 0)
-		(color 0 0 0 0)
-	)
-	(junction
 		(at 181.61 25.4)
 		(diameter 0)
@@
 	)
 	(junction
-		(at 237.49 119.38)
-		(diameter 0)
-		(color 0 0 0 0)
-	)
-	(junction
 		(at 16.51 22.86)
 		(diameter 0)
@@
 	)
 	(junction
+		(at 237.49 102.87)
+		(diameter 0)
+		(color 0 0 0 0)
+	)
+	(junction
 		(at 162.56 77.47)
 		(diameter 0)
@@
 	)
 	(junction
+		(at 237.49 119.38)
+		(diameter 0)
+		(color 0 0 0 0)
+	)
+	(junction
 		(at 116.84 77.47)
 		(diameter 0)
@@
 	(wire
 		(pts
-			(xy 237.49 102.87) (xy 245.11 102.87)
-		)
-		(stroke
-			(width 0)
-			(type default)
-		)
-	)
-	(wire
-		(pts
 			(xy 260.35 111.76) (xy 260.35 110.49)
 		)
@@
 	(wire
 		(pts
+			(xy 237.49 102.87) (xy 245.11 102.87)
+		)
+		(stroke
+			(width 0)
+			(type default)
+		)
+	)
+	(wire
+		(pts
 			(xy 113.03 146.05) (xy 120.65 146.05)
 		)
@@
 	(wire
 		(pts
-			(xy 237.49 119.38) (xy 261.62 119.38)
-		)
-		(stroke
-			(width 0)
-			(type default)
-		)
-	)
-	(wire
-		(pts
 			(xy 132.08 48.26) (xy 147.32 48.26)
 		)
@@
 	(wire
 		(pts
+			(xy 237.49 119.38) (xy 261.62 119.38)
+		)
+		(stroke
+			(width 0)
+			(type default)
+		)
+	)
+	(wire
+		(pts
 			(xy 114.3 29.21) (xy 114.3 36.83)
 		)
@@
 			)
 		)
-		(property "Value" "OPT"
+		(property "Value" "TBD"
 			(at 186.69 130.81 90)
 			(show_name no)
